Commit message: Update controller

File: description/robot_core.xacro (robot description, xacro)
@@ -1,19 +1,4 @@
 <?xml version="1.0"?>
 <robot xmlns:xacro="http://www.ros.org/wiki/xacro" >
-    <!-- <xacro:property name="chassis_length" value="1.230"/>
-    <xacro:property name="chassis_width" value="0.610"/>
-    <xacro:property name="chassis_height" value="0.360"/>
-    <xacro:property name="chassis_mass" value="70.0"/>
-    <xacro:property name="wheel_radius" value="0.180"/>
-    <xacro:property name="wheel_thickness" value="0.140"/>
-    <xacro:property name="wheel_mass" value="1.0"/>
-    <xacro:property name="wheel_offset_x" value="0.16"/>
-    <xacro:property name="wheel_offset_y" value="0.410"/>
-    <xacro:property name="wheel_offset_z" value="-0.035"/>
-    <xacro:property name="caster_wheel_radius" value="0.105"/>
-    <xacro:property name="caster_wheel_mass" value="0.25"/>
-    <xacro:property name="caster_wheel_offset_x" value="1.120"/>
-    <xacro:property name="caster_wheel_offset_y" value="0.245"/>
-    <xacro:property name="caster_wheel_offset_z" value="-0.140"/> -->
   <!-- Define robot constants -->
   <xacro:property name="base_width" value="0.610"/>
@@ -71,5 +56,4 @@
   <!-- Robot Footprint -->
   <link name="base_footprint">
-    <xacro:box_inertia m="0" w="0" d="0" h="0"/>
   </link>
   <joint name="base_joint" type="fixed">
